Commit message: Comments, removed empty lines

File: src/base/robot_desc/inertial_macros.xacro (robot description, xacro)
@@ -1,5 +1,4 @@
 <?xml version="1.0"?>
 <robot xmlns:xacro="http://www.ros.org/wiki/xacro">
-    <!-- INERTIAL MACROS -->
     <xacro:macro name="inertial_box" params="mass x y z *origin">
       <inertial>

File: src/base/robot_desc/swervebot.xacro (robot description, xacro)
@@ -1,4 +1,5 @@
 <?xml version="1.0"?>
 <robot name="swervebot" xmlns:xacro="http://www.ros.org/wiki/xacro">
+    <!-- Master xacro file -->
     <xacro:include filename="inertial_macros.xacro"/>
     <xacro:include filename="materials.xacro"/>

File: src/base/robot_desc/swervebot_car.xacro (robot description, xacro)
@@ -23,5 +23,5 @@
         </xacro:inertial_box>
     </link>
-    <!-- ALERT: This joint is not accurately positioned at the wheel contact to the ground -->
+    <!-- WARNING: This joint is not accurately positioned at the wheel contact to the ground -->
     <joint name="base_footprint_joint" type="fixed">
         <parent link="base_footprint_link"/>
@@ -29,5 +29,5 @@
         <origin xyz="0 0 ${frame_depth * 1.5 + set_wheel_radius}"/>
     </joint>
-    <!-- BUMPERS -->
+    <!-- BUMPER LINKS -->
     <xacro:property name="bumper_thick_x" value="${frame_length / 10}"/>
     <xacro:property name="bumper_length_x" value="${frame_width / 1.8}"/>
@@ -99,4 +99,5 @@
         </xacro:inertial_box>
     </link>
+    <!-- GENERATE SWERVE WHEEL LINKS AND JOINTS -->
     <xacro:include filename="swervebot_wheel.xacro"/>
     <xacro:swerve_wheel name="front_left" radius="${set_wheel_radius}" rotater_material="darkgray" spinner_material="black"/>

File: src/base/robot_desc/swervebot_wheel.xacro (robot description, xacro)
@@ -1,16 +1,10 @@
 <?xml version="1.0"?>
 <robot xmlns:xacro="http://www.ros.org/wiki/xacro">
-    <!-- DIFFERENTIAL SWERVE WHEEL MACRO -->
+    <!--
+        This macro generate two links representing the wheel and differential drive
+        gear mechanism and make a joint out of them.
+     -->
     <xacro:macro name="swerve_wheel" params="name radius rotater_material spinner_material">
         <xacro:property name="wheel_radius" value="${radius}"/>
-        <!-- Uncomment this and its joint to rotater to find out the front face of the wheel -->
-        <!-- <link name="${name}_frontmark_link">
-            <visual>
-                <geometry>
-                    <box size="${wheel_radius * 0.5} ${wheel_radius * 1.5} ${wheel_radius * 0.5}"/>
-                </geometry>
-                <material name="${rotater_material}"/>
-            </visual>
-        </link> -->
         <link name="${name}_rotater_link">
             <visual>
@@ -51,9 +45,4 @@
             <axis xyz="0 0 1"/>
         </joint>
-        <!-- <joint name="${name}_frontmark_joint" type="fixed">
-            <origin xyz="${wheel_radius * -1.25} 0 0"/>
-            <parent link="${name}_rotater_link"/>
-            <child link="${name}_frontmark_link"/>
-        </joint> -->
     </xacro:macro>
 </robot>
